File: Block-JAN6418.kicad_sch (KiCad schematic)
At the start: 17 parts, among them J1 B+, J2 Sig_gnd, J3 Sig_in, J4 Sig_out, J5 9V, U1 JAN6418, U2 LM317L

Commit message: generate drl, grbrs, update sch from pcb
Parts:
- renumbered J5 to +9V, J1 to B+, R6 to Impedance, R3 to Ra, J2 to Sig_gnd, J3 to Sig_in, J4 to Sig_out
Changed lines of the file:
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@@
 		(dnp no)
 		(fields_autoplaced yes)
-		(property "Reference" "J3"
+		(property "Reference" "Sig_in"
 			(at 20.32 54.61 0)
 			(effects
@@
 			(project "Block-JAN6418"
 				(path "/3c383edb-2f76-4d07-a4e0-15afb529fb0e"
-					(reference "J3")
+					(reference "Sig_in")
 					(unit 1)
 				)
@@
 		(dnp no)
 		(fields_autoplaced yes)
-		(property "Reference" "R3"
+		(property "Reference" "Ra"
 			(at 52.07 30.4799 0)
 			(effects
@@
 			(project ""
 				(path "/3c383edb-2f76-4d07-a4e0-15afb529fb0e"
-					(reference "R3")
+					(reference "Ra")
 					(unit 1)
 				)
@@
 		(dnp no)
 		(fields_autoplaced yes)
-		(property "Reference" "J4"
+		(property "Reference" "Sig_out"
 			(at 71.12 39.3699 0)
 			(effects
@@
 			(project "Block-JAN6418"
 				(path "/3c383edb-2f76-4d07-a4e0-15afb529fb0e"
-					(reference "J4")
+					(reference "Sig_out")
 					(unit 1)
 				)
@@
 		(dnp no)
 		(fields_autoplaced yes)
-		(property "Reference" "R6"
+		(property "Reference" "Impedance"
 			(at 39.37 67.3099 0)
 			(effects
@@
 			(project "Block-JAN6418"
 				(path "/3c383edb-2f76-4d07-a4e0-15afb529fb0e"
-					(reference "R6")
+					(reference "Impedance")
 					(unit 1)
 				)
@@
 		(dnp no)
 		(fields_autoplaced yes)
-		(property "Reference" "J1"
+		(property "Reference" "B+"
 			(at 52.07 17.7799 90)
 			(effects
@@
 			(project ""
 				(path "/3c383edb-2f76-4d07-a4e0-15afb529fb0e"
-					(reference "J1")
+					(reference "B+")
 					(unit 1)
 				)
@@
 		(dnp no)
 		(fields_autoplaced yes)
-		(property "Reference" "J5"
+		(property "Reference" "+9V"
 			(at 20.32 17.78 0)
 			(effects
@@
 			(project "Block-JAN6418"
 				(path "/3c383edb-2f76-4d07-a4e0-15afb529fb0e"
-					(reference "J5")
+					(reference "+9V")
 					(unit 1)
 				)
@@
 		(dnp no)
 		(fields_autoplaced yes)
-		(property "Reference" "J2"
+		(property "Reference" "Sig_gnd"
 			(at 22.86 34.2899 90)
 			(effects
@@
 			(project "Block-JAN6418"
 				(path "/3c383edb-2f76-4d07-a4e0-15afb529fb0e"
-					(reference "J2")
-					(unit 1)
-				)
+					(reference "Sig_gnd")
+					(unit 1)
+				)
